File: BLLED.kicad_pcb (KiCad board)
At the start: 2 copper layers, 28 x 51.5 mm, 11 parts, among them J1 LEDs, J2 5V Input, J3 P1S, Q1 IRLB8721

Commit message: update pcb
Parts:
- J1, J3: footprint TerminalBlock_RND:TerminalBlock_RND_205-00276_1x02_P5.00mm_Vertical -> TerminalBlock:TerminalBlock_bornier-2_P5.08mm
- J2: value 5V Input -> Input; footprint TerminalBlock_RND:TerminalBlock_RND_205-00276_1x02_P5.00mm_Vertical -> TerminalBlock:TerminalBlock_bornier-2_P5.08mm
- moved J3 2.83 mm to (114.2, 69.3)
- moved J1 2.78 mm to (114.2, 57.9)
- moved J2 1.83 mm to (125.8, 62.9)
- moved R1 1.49 mm to (120.9, 69.4)
- moved R2 1.49 mm to (131.1, 74.4)
Connections:
- net /GND renamed GND
Routing:
- net GND: track 124.6 -> 0.00 mm
- net Net-(J1-Pin_2): track 20.1 -> 26.4 mm
- net Net-(J1-Pin_1): track 9.07 -> 13.7 mm, vias 0 -> 1
- net Net-(J3-Pin_1): track 17.7 -> 19.0 mm
- net Net-(Q1-G): track 19.6 -> 18.9 mm
- added copper zone on B.Cu, net GND
